Commit message: Rename URDF file

File: description/V6_snake_URDF/urdf/V6_snake_URDF.urdf (robot description, URDF)
Before this commit: robot B_snake_URDF.SLDASM, 9 links, 8 joints
Links:
- link base_link: mass 0.0014137 -> 0.00141371669411541; geometry collision mesh filename=package://V6_snake_URDF/meshes/base_link.STL; visual mesh filename=package://V6_snake_URDF/meshes/base_link.STL
- link elbow_link: mass 0.00011415 -> 0.000114145071751143; geometry collision mesh filename=package://V6_snake_URDF/meshes/elbow_link.STL; visual mesh filename=package://V6_snake_URDF/meshes/elbow_link.STL
- link forearm_link: mass 0.00027925 -> 0.000279249014923545; geometry collision mesh filename=package://V6_snake_URDF/meshes/forearm_link.STL; visual mesh filename=package://V6_snake_URDF/meshes/forearm_link.STL
- link gripper_1: mass 9.5944E-05 -> 9.59439630385687E-05; geometry collision mesh filename=package://V6_snake_URDF/meshes/gripper_1.STL; visual mesh filename=package://V6_snake_URDF/meshes/gripper_1.STL
- link gripper_2: geometry collision mesh filename=package://V6_snake_URDF/meshes/gripper_2.STL; visual mesh filename=package://V6_snake_URDF/meshes/gripper_2.STL
- link hand_link: mass 0.00040496 -> 0.000404964898437663; geometry collision mesh filename=package://V6_snake_URDF/meshes/hand_link.STL; visual mesh filename=package://V6_snake_URDF/meshes/hand_link.STL
- link shoulder_link: mass 0.00011415 -> 0.000114145071751143; geometry collision mesh filename=package://V6_snake_URDF/meshes/shoulder_link.STL; visual mesh filename=package://V6_snake_URDF/meshes/shoulder_link.STL
- link snake_start_link: mass 0.00071324 -> 0.000713238856062597; geometry collision mesh filename=package://V6_snake_URDF/meshes/snake_start_link.STL; visual mesh filename=package://V6_snake_URDF/meshes/snake_start_link.STL
- link upperarm_link: mass 0.00066722 -> 0.000667220219941384; geometry collision mesh filename=package://V6_snake_URDF/meshes/upperarm_link.STL; visual mesh filename=package://V6_snake_URDF/meshes/upperarm_link.STL
Joints:
- joint elbow_joint_dist: origin xyz=0 0 0.005 rpy=0 0 3.1416 -> xyz=0 0 0.00500000000000002 rpy=0 0 3.14159265358979
- joint gripper_2: origin xyz=0 0 0.019 rpy=0.3293 0 3.1416 -> xyz=0 0 0.019 rpy=0.329304747776595 0 3.14159265358979
- joint gripper_joint_1: origin xyz=0 0 0.019 rpy=0.3293 0 0 -> xyz=0 0 0.019 rpy=0.329304747776595 0 0
- joint shoulder_joint_dist: origin xyz=0 0 0.005 rpy=0 0 -3.1416 -> xyz=0 0 0.005 rpy=0 0 -3.14159265358979

Commit message: Fix urdf file. Update README

File: description/V6_snake_URDF/urdf/V6_snake_URDF.urdf (robot description, URDF)
Before this commit: robot V6_snake_URDF, 9 links, 8 joints
Links:
- link base_link: geometry collision mesh filename=file:///home/dingkun/ros2_ws/src/s_bot_ros2/description/V6_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; visual mesh filename=file:///home/dingkun/ros2_ws/src/s_bot_ros2/description/V6_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
- link elbow_link: geometry collision mesh filename=file:///home/dingkun/ros2_ws/src/s_bot_ros2/description/V6_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; visual mesh filename=file:///home/dingkun/ros2_ws/src/s_bot_ros2/description/V6_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
- link forearm_link: geometry collision mesh filename=file:///home/dingkun/ros2_ws/src/s_bot_ros2/description/V6_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; visual mesh filename=file:///home/dingkun/ros2_ws/src/s_bot_ros2/description/V6_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
- link gripper_1: geometry collision mesh filename=file:///home/dingkun/ros2_ws/src/s_bot_ros2/description/V6_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; visual mesh filename=file:///home/dingkun/ros2_ws/src/s_bot_ros2/description/V6_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
- link gripper_2: geometry collision mesh filename=file:///home/dingkun/ros2_ws/src/s_bot_ros2/description/V6_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; visual mesh filename=file:///home/dingkun/ros2_ws/src/s_bot_ros2/description/V6_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
- link hand_link: geometry collision mesh filename=file:///home/dingkun/ros2_ws/src/s_bot_ros2/description/V6_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; visual mesh filename=file:///home/dingkun/ros2_ws/src/s_bot_ros2/description/V6_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
- link shoulder_link: geometry collision mesh filename=file:///home/dingkun/ros2_ws/src/s_bot_ros2/description/V6_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; visual mesh filename=file:///home/dingkun/ros2_ws/src/s_bot_ros2/description/V6_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
- link snake_start_link: geometry collision mesh filename=file:///home/dingkun/ros2_ws/src/s_bot_ros2/description/V6_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; visual mesh filename=file:///home/dingkun/ros2_ws/src/s_bot_ros2/description/V6_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
- link upperarm_link: geometry collision mesh filename=file:///home/dingkun/ros2_ws/src/s_bot_ros2/description/V6_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; visual mesh filename=file:///home/dingkun/ros2_ws/src/s_bot_ros2/description/V6_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
Joints:
- joint elbow_joint_dist: limit lower=0 upper=0.785 effort=1 velocity=1 -> lower=-0.785 upper=0 effort=1 velocity=1
- joint gripper_2: limit lower=0 upper=0.785 effort=1 velocity=1 -> lower=-0.785 upper=0 effort=1 velocity=1
- joint gripper_joint_1: limit lower=-0.785 upper=0 effort=1 velocity=1 -> lower=0 upper=0.785 effort=1 velocity=1
- joint shoulder_joint_dist: limit lower=0 upper=0.785 effort=1 velocity=1 -> lower=-0.785 upper=0 effort=1 velocity=1
